Commit message: Changed urdf to RILAB's canine

File: rsc/urdf/canine/urdf/canine_RILAB.urdf (robot description, URDF)
Before this commit: robot canineV5_wheeled, 14 links, 13 joints
Links:
- link FL_calf: geometry collision sphere radius=0.025; visual mesh filename=../meshes/HR_calf_1.stl scale=0.001 0.001 0.001
- link FL_hip: mass 0.7498 -> 0.8848
- link FR_calf: geometry collision sphere radius=0.025; visual mesh filename=../meshes/HR_calf_1.stl scale=0.001 0.001 0.001
- link FR_hip: mass 0.7498 -> 0.8848
- link HL_calf: geometry collision sphere radius=0.025; visual mesh filename=../meshes/HR_calf_1.stl scale=0.001 0.001 0.001
- link HL_hip: mass 0.7498 -> 0.8848
- link HR_calf: geometry collision sphere radius=0.025; visual mesh filename=../meshes/HR_calf_1.stl scale=0.001 0.001 0.001
- link HR_hip: mass 0.7498 -> 0.8848
- link trunk: mass 9.7728 -> 10.3128
Joints:
- joint FL_HIP: limit lower=-1.8 upper=1.8 effort=30 velocity=13.0 -> (none); origin xyz=0.1855 0.075 0.0 rpy=0 0 0 -> xyz=0.1935 0.075 0.0 rpy=0 0 0
- joint FL_KNEE: limit lower=-3.14 upper=0.0 effort=30 velocity=13.0 -> (none)
- joint FL_THIGH: limit lower=-3.14 upper=1.8 effort=30 velocity=13.0 -> (none)
- joint FR_HIP: limit lower=-1.8 upper=1.8 effort=30 velocity=13.0 -> (none); origin xyz=0.1855 -0.075 0.0 rpy=0 0 0 -> xyz=0.1935 -0.075 0.0 rpy=0 0 0
- joint FR_KNEE: limit lower=-3.14 upper=0.0 effort=30 velocity=13.0 -> (none)
- joint FR_THIGH: limit lower=-3.14 upper=1.8 effort=30 velocity=13.0 -> (none)
- joint HL_HIP: limit lower=-1.8 upper=1.8 effort=30 velocity=13.0 -> (none); origin xyz=-0.1855 0.075 0.0 rpy=0 0 0 -> xyz=-0.1935 0.075 0.0 rpy=0 0 0
- joint HL_KNEE: limit lower=-3.14 upper=0.0 effort=30 velocity=13.0 -> (none)
- joint HL_THIGH: limit lower=-3.14 upper=1.8 effort=30 velocity=13.0 -> (none)
- joint HR_HIP: limit lower=-1.8 upper=1.8 effort=30 velocity=13.0 -> (none); origin xyz=-0.1855 -0.075 0.0 rpy=0 0 0 -> xyz=-0.1935 -0.075 0.0 rpy=0 0 0
- joint HR_KNEE: limit lower=-3.14 upper=0.0 effort=30 velocity=13.0 -> (none)
- joint HR_THIGH: limit lower=-3.14 upper=1.8 effort=30 velocity=13.0 -> (none)

Commit message: Updated urdf

File: rsc/urdf/canine/urdf/canine_RILAB.urdf (robot description, URDF)
Before this commit: robot canine_RILAB, 14 links, 13 joints
Links:
- link FL_calf: mass 0.268 -> 0.223676
- link FL_hip: mass 0.8848 -> 0.996202
- link FL_thigh: mass 1.539 -> 1.400484
- link FR_calf: mass 0.268 -> 0.223676
- link FR_hip: mass 0.8848 -> 0.996202
- link FR_thigh: mass 1.539 -> 1.400484
- link HL_calf: mass 0.268 -> 0.223676
- link HL_hip: mass 0.8848 -> 0.996202
- link HL_thigh: mass 1.539 -> 1.400484
- link HR_calf: mass 0.268 -> 0.223676
- link HR_hip: mass 0.8848 -> 0.996202
- link HR_thigh: mass 1.539 -> 1.400484
- link trunk: mass 10.3128 -> 11.9704
